Commit message: Balance legs and made FT sensors at joints working

File: ros2/src/huron_description/urdf/huron_inertia.xacro (robot description, xacro)
@@ -50,5 +50,5 @@
     <xacro:macro name="insert_inertia_l_hip_yaw_link">
       <origin
-        xyz="0.00063365 -0.00053469 0.063496"
+        xyz="0.00063365 -0.00053469 0.063505"
         rpy="0 0 0" />
       <mass

File: ros2/src/huron_description/urdf/huron_left_leg.xacro (robot description, xacro)
@@ -5,7 +5,7 @@
     <xacro:macro name="huron_left_leg" params="parent dxl_effort dxl_speed">
         <!-- left hip yaw joint -->
-        <joint name="l_hip_yaw_joint" type="fixed">
-          <origin
-            xyz="-0.0775 0 -0.1451242"
+        <joint name="l_hip_yaw_joint" type="revolute">
+          <origin
+            xyz="-0.0775 0 -0.14512"
             rpy="0 0 0" />
           <parent link="${parent}" />
@@ -37,5 +37,5 @@
         <joint
           name="l_hip_roll_joint"
-          type="fixed">
+          type="revolute">
           <origin
             xyz="0 0 0"

File: ros2/src/huron_description/urdf/huron_right_leg.xacro (robot description, xacro)
@@ -7,5 +7,5 @@
         <joint
           name="r_hip_yaw_joint"
-          type="fixed">
+          type="revolute">
           <origin
             xyz="0.0775 0 -0.14512"
@@ -42,5 +42,5 @@
         <joint
           name="r_hip_roll_joint"
-          type="fixed">
+          type="revolute">
           <origin
             xyz="0 0 0"

File: ros2/src/huron_gazebo/urdf/huron.xacro (robot description, xacro)
@@ -41,8 +41,13 @@
     <gazebo>
     <plugin name="r1_ft_sensor" filename="libgazebo_ros_ft_sensor.so">
-        <updateRate>100.0</updateRate>
-        <topicName>/huron/sensor/r1_ft_sensor</topicName>
-        <jointName>r_ankle_roll_joint</jointName>
-        <gaussianNoise>0.0</gaussianNoise>
+      <ros>
+        <namespace>/huron/sensor</namespace>
+        <remapping>wrench:=r1_ft_sensor</remapping>
+      </ros>
+      <update_rate>100</update_rate>
+      <!-- <body_name>r_ankle_roll_link</body_name> -->
+      <!-- <frame_name>r_ankle_roll_link</frame_name> -->
+      <joint_name>r_ankle_roll_joint</joint_name>
+      <gaussian_noise>0.0</gaussian_noise>
     </plugin>
     </gazebo>
@@ -52,22 +57,27 @@
     <gazebo>
     <plugin name="l1_ft_sensor" filename="libgazebo_ros_ft_sensor.so">
-        <updateRate>100.0</updateRate>
-        <topicName>/huron/sensor/l1_ft_sensor</topicName>
-        <jointName>l_ankle_roll_joint</jointName>
-        <gaussianNoise>0.0</gaussianNoise>
+      <ros>
+        <namespace>/huron/sensor</namespace>
+        <remapping>wrench:=l1_ft_sensor</remapping>
+      </ros>
+      <update_rate>100</update_rate>
+      <!-- <body_name>l_ankle_roll_link</body_name> -->
+      <!-- <frame_name>l_ankle_roll_link</frame_name> -->
+      <joint_name>l_ankle_roll_joint</joint_name>
+      <gaussian_noise>0.0</gaussian_noise>
     </plugin>
     </gazebo>
-    <gazebo reference = "l_hip_yaw_joint">
-    	<preserveFixedJoint>true</preserveFixedJoint>
-    </gazebo>
-    <gazebo reference = "l_hip_roll_joint">
-    	<preserveFixedJoint>true</preserveFixedJoint>
-    </gazebo>
-    <gazebo reference = "r_hip_yaw_joint">
-    	<preserveFixedJoint>true</preserveFixedJoint>
-    </gazebo>
-    <gazebo reference = "r_hip_roll_joint">
-    	<preserveFixedJoint>true</preserveFixedJoint>
-    </gazebo>
+    <!-- <gazebo reference = "l_hip_yaw_joint"> -->
+    <!-- 	<preserveFixedJoint>true</preserveFixedJoint> -->
+    <!-- </gazebo> -->
+    <!-- <gazebo reference = "l_hip_roll_joint"> -->
+    <!-- 	<preserveFixedJoint>true</preserveFixedJoint> -->
+    <!-- </gazebo> -->
+    <!-- <gazebo reference = "r_hip_yaw_joint"> -->
+    <!-- 	<preserveFixedJoint>true</preserveFixedJoint> -->
+    <!-- </gazebo> -->
+    <!-- <gazebo reference = "r_hip_roll_joint"> -->
+    <!-- 	<preserveFixedJoint>true</preserveFixedJoint> -->
+    <!-- </gazebo> -->
     <!-- <gazebo reference = "dummy_joint"> -->
     <!-- 	<preserveFixedJoint>true</preserveFixedJoint> -->
