Commit message: Factor huron_description
This commit separates pure URDF descriptionn from Gazebo-specific config.
The robot generation is now also a macro (huron_base), which can be re-used
in different xacro files.

File: ros2/src/huron_description/urdf/huron.xacro (robot description, xacro)
@@ -1,83 +1,9 @@
 <?xml version="1.0"?>
-<robot name="huron"
-    xmlns:xacro="http://www.ros.org/wiki/xacro">
-    <!-- <xacro:property name="pi" value="3.141592654"/> -->
-    <!-- Import xacro file -->
-    <xacro:include filename="$(find huron_description)/urdf/materials.xacro" />
-    <xacro:include filename="$(find huron_description)/urdf/huron_visuals.xacro" />
-    <xacro:include filename="$(find huron_description)/urdf/huron_inertia.xacro" />
-    <xacro:include filename="$(find huron_description)/urdf/huron_transmissions.xacro" />
-    <xacro:include filename="$(find huron_description)/urdf/huron_right_leg.xacro" />
-    <xacro:include filename="$(find huron_description)/urdf/huron_left_leg.xacro" />
-    <xacro:include filename="$(find huron_description)/urdf/huron_misc.xacro" />
-    <xacro:include filename="$(find huron_description)/urdf/huron_gazebo.xacro" />
-    <xacro:include filename="$(find huron_description)/urdf/huron_ros2_control.xacro" />
-    <!-- Used for fixing robot -->
-    <!--<link name="world"></link>
-    <joint name="world_fixed" type="fixed">
-        <origin xyz="0 0 0.764" rpy="0 0 0"/>
-        <parent link="world"/>
-        <child link="base_link"/>
-    </joint> -->
-    <link name="dummy"></link>
-    <link name="base_link">
-        <visual>
-            <origin xyz="0 0 0" rpy="0 0 0" />
-            <geometry>
-                <mesh filename="package://huron_description/meshes/base_link.STL" scale="1 1 1" />
-            </geometry>
-        </visual>
-        <collision>
-            <origin xyz="0 0 0" rpy="0 0 0" />
-            <geometry>
-                <mesh filename="package://huron_description/meshes/base_link.STL" scale="1 1 1" />
-            </geometry>
-        </collision>
-        <inertial>
-          <origin
-            xyz="-1.3585E-07 5.07E-07 0.026975"
-            rpy="0 0 0" />
-          <mass
-            value="3.4072" />
-          <inertia
-            ixx="0.00319"
-            ixy="-1.7776E-09"
-            ixz="-1.7316E-09"
-            iyy="0.010531"
-            iyz="6.4623E-09"
-            izz="0.012315" />
-        </inertial>
-    </link>
-    <joint name="dummy_joint" type="fixed">
-        <parent link="dummy"/>
-        <child link="base_link"/>
-    </joint>
-    <!-- <joint name="base_fixed" type="fixed"> -->
-    <!--     <origin xyz="0 0 0" rpy="0 0 0"/> -->
-    <!--     <parent link="base_link"/> -->
-    <!--     <child link="base_footprint"/> -->
-    <!-- </joint> -->
-    <!-- <link name="base_footprint"> -->
-    <!--     <visual> -->
-    <!--         <xacro:insert_mesh_base_link /> -->
-    <!--     </visual> -->
-    <!--     <collision> -->
-    <!--         <xacro:insert_mesh_base_link /> -->
-    <!--     </collision> -->
-    <!--     <inertial> -->
-    <!--         <xacro:insert_inertia_base_link /> -->
-    <!--     </inertial> -->
-    <!-- </link> -->
-    <!-- imu joint -->
-    <joint name="imu_fixed" type="fixed">
-        <origin xyz="0 0 0" rpy="0 0 0"/>
-        <parent link="base_link"/>
-        <child link="imu_link"/>
-    </joint>
-    <link name="imu_link"></link>
-    <!-- leg link -->
-    <xacro:huron_right_leg parent="base_link" dxl_effort="1000000" dxl_speed="3000"/>
-    <xacro:huron_left_leg parent="base_link" dxl_effort="1000000" dxl_speed="3000"/>
-    <xacro:huron_misc />
-    <xacro:huron_ros2_control name="huron" prefix="" />
+<robot name="huron" xmlns:xacro="http://www.ros.org/wiki/xacro">
+  <!--
+    Top level description file for HURON. This can be used to generate a URDF.
+  -->
+  <xacro:include filename="$(find huron_description)/urdf/huron_macro.xacro" />
+  <!-- Add HURON Base -->
+  <xacro:huron_base />
 </robot>

File: ros2/src/huron_gazebo/urdf/huron.xacro (robot description, xacro)
@@ -1,11 +1,11 @@
 <?xml version="1.0"?>
-<robot
-    xmlns:xacro="http://www.ros.org/wiki/xacro">
-    <!-- ros_control plugin -->
-    <gazebo>
-        <plugin name="gazebo_ros_control" filename="libgazebo_ros_control.so">
-            <robotNamespace>/huron</robotNamespace>
-         </plugin>
-    </gazebo>
+<robot xmlns:xacro="http://www.ros.org/wiki/xacro" name="huron">
+    <!-- HURON model for use with Gazebo simulation -->
+    <xacro:include filename="$(find huron_description)/urdf/huron_macro.xacro" />
+    <xacro:include filename="$(find huron_gazebo)/urdf/huron_ros2_control.xacro" />
+    <!-- Add HURON Base -->
+    <xacro:huron_base />
+    <!-- ros2_control plugin -->
+    <xacro:huron_ros2_control name="huron" prefix="" />
     <gazebo>
         <plugin name="ground_truth" filename="libgazebo_ros_p3d.so">

File: ros2/src/huron_gazebo/urdf/huron_ros2_control.xacro (robot description, xacro)
@@ -3,10 +3,4 @@
   <xacro:macro name="huron_ros2_control" params="name prefix">
     <ros2_control name="${name}" type="system">
-      <!-- <hardware>
-        <plugin>ros2_control_demo_hardware/RRBotSystemPositionOnlyHardware</plugin>
-        <param name="example_param_hw_start_duration_sec">0</param>
-        <param name="example_param_hw_stop_duration_sec">3.0</param>
-        <param name="example_param_hw_slowdown">100</param>
-      </hardware> -->
       <hardware>
           <plugin>gazebo_ros2_control/GazeboSystem</plugin>
@@ -123,5 +117,5 @@
     <gazebo>
         <plugin filename="libgazebo_ros2_control.so" name="gazebo_ros2_control">
-          <parameters>$(find huron_control)/config/gazebo_controllers.yaml</parameters>
+          <parameters>$(find huron_gazebo)/config/gazebo_controllers.yaml</parameters>
         </plugin>
       </gazebo>

Commit message: URDF for HURON with FSR

File: ros2/src/huron_description/urdf/huron.xacro (robot description, xacro)
@@ -1,9 +1,16 @@
 <?xml version="1.0"?>
 <robot name="huron" xmlns:xacro="http://www.ros.org/wiki/xacro">
-  <!--
-    Top level description file for HURON. This can be used to generate a URDF.
-  -->
-  <xacro:include filename="$(find huron_description)/urdf/huron_macro.xacro" />
-  <!-- Add HURON Base -->
-  <xacro:huron_base />
+    <xacro:arg name="force_sensor" default="ft_sensor" />
+    <xacro:property name="force_sensor_prop" value="$(arg force_sensor)" />
+    <!--
+      Top level description file for HURON. This can be used to generate a URDF for non-simulation applications.
+      URDF generation syntax:
+        ros2 run xacro xacro huron.urdf [ft_sensor:=<ft_sensor|fsr>]
+    -->
+    <xacro:include filename="$(find huron_description)/urdf/huron_macro.xacro" />
+    <xacro:if value="${force_sensor_prop == 'fsr'}">
+        <xacro:include filename="$(find huron_description)/urdf/huron_fsr.xacro" />
+    </xacro:if>
+    <!-- Add HURON Base -->
+    <xacro:huron_base />
 </robot>

File: ros2/src/huron_gazebo/urdf/huron.xacro (robot description, xacro)
@@ -1,4 +1,6 @@
 <?xml version="1.0"?>
 <robot xmlns:xacro="http://www.ros.org/wiki/xacro" name="huron">
+    <xacro:arg name="force_sensor" default="ft_sensor" />
+    <xacro:property name="force_sensor_prop" value="$(arg force_sensor)" />
     <!-- HURON model for use with Gazebo simulation -->
     <xacro:include filename="$(find huron_description)/urdf/huron_macro.xacro" />
@@ -36,51 +38,10 @@
         </sensor>
     </gazebo>
-    <gazebo reference ="r_ankle_roll_joint">
-    	<provideFeedback>true</provideFeedback>
-    </gazebo>
-    <gazebo>
-    <plugin name="r1_ft_sensor" filename="libgazebo_ros_ft_sensor.so">
-      <ros>
-        <namespace>/huron/sensor</namespace>
-        <remapping>wrench:=r1_ft_sensor</remapping>
-      </ros>
-      <update_rate>100</update_rate>
-      <!-- <body_name>r_ankle_roll_link</body_name> -->
-      <!-- <frame_name>r_ankle_roll_link</frame_name> -->
-      <joint_name>r_ankle_roll_joint</joint_name>
-      <gaussian_noise>0.0</gaussian_noise>
-    </plugin>
-    </gazebo>
-    <gazebo reference ="l_ankle_roll_joint">
-    	<provideFeedback>true</provideFeedback>
-    </gazebo>
-    <gazebo>
-    <plugin name="l1_ft_sensor" filename="libgazebo_ros_ft_sensor.so">
-      <ros>
-        <namespace>/huron/sensor</namespace>
-        <remapping>wrench:=l1_ft_sensor</remapping>
-      </ros>
-      <update_rate>100</update_rate>
-      <!-- <body_name>l_ankle_roll_link</body_name> -->
-      <!-- <frame_name>l_ankle_roll_link</frame_name> -->
-      <joint_name>l_ankle_roll_joint</joint_name>
-      <gaussian_noise>0.0</gaussian_noise>
-    </plugin>
-    </gazebo>
-    <!-- <gazebo reference = "l_hip_yaw_joint"> -->
-    <!-- 	<preserveFixedJoint>true</preserveFixedJoint> -->
-    <!-- </gazebo> -->
-    <!-- <gazebo reference = "l_hip_roll_joint"> -->
-    <!-- 	<preserveFixedJoint>true</preserveFixedJoint> -->
-    <!-- </gazebo> -->
-    <!-- <gazebo reference = "r_hip_yaw_joint"> -->
-    <!-- 	<preserveFixedJoint>true</preserveFixedJoint> -->
-    <!-- </gazebo> -->
-    <!-- <gazebo reference = "r_hip_roll_joint"> -->
-    <!-- 	<preserveFixedJoint>true</preserveFixedJoint> -->
-    <!-- </gazebo> -->
-    <!-- <gazebo reference = "dummy_joint"> -->
-    <!-- 	<preserveFixedJoint>true</preserveFixedJoint> -->
-    <!-- </gazebo> -->
+    <xacro:if value="${force_sensor_prop == 'fsr'}">
+        <xacro:include filename="$(find huron_gazebo)/urdf/huron_fsr.xacro" />
+    </xacro:if>
+    <xacro:if value="${force_sensor_prop == 'ft_sensor'}">
+        <xacro:include filename="$(find huron_gazebo)/urdf/huron_ft_sensor.xacro" />
+    </xacro:if>
     <!-- World -->
     <gazebo reference="world"></gazebo>
